Commit message: adding content 20231108

File: src/dofbot_moveit/urdf/dofbot.urdf (robot description, URDF)
Before this commit: robot dofbot, 6 links, 5 joints
Joints:
- joint joint1: limit lower=-1.5708 upper=1.5708 effort=30 velocity=1.0 -> lower=-1.5708 upper=1.5708 effort=30.0 velocity=1.5
- joint joint2: limit lower=-1.5708 upper=1.5708 effort=30 velocity=1.0 -> lower=-1.5708 upper=1.5708 effort=30.0 velocity=1.5
- joint joint3: limit lower=-1.5708 upper=1.5708 effort=30 velocity=1.0 -> lower=-1.5708 upper=1.5708 effort=30.0 velocity=1.5
- joint joint4: limit lower=-1.5708 upper=1.5708 effort=30 velocity=1.0 -> lower=-1.5708 upper=1.5708 effort=30.0 velocity=1.5
- joint joint5: limit lower=-1.5708 upper=3.1416 effort=30 velocity=1.0 -> lower=-1.5708 upper=3.1416 effort=30.0 velocity=1.5
