Commit message: adding conteng 20231119

File: src/dofbot_description/urdf/dofbot.urdf.xacro (robot description, xacro)
@@ -2,5 +2,4 @@
 <robot xmlns:xacro="http://wiki.ros.org/xacro" name="dofbot">
     <xacro:include filename="$(find dofbot_description)/urdf/dofbot_description.urdf.xacro"/>
-    <link name="world"/>
     <xacro:dof6bot_description/>
     <xacro:include filename="$(find dofbot_description)/urdf/dofbot.ros2_control.xacro"/>

File: src/dofbot_description/urdf/dofbot_description.urdf.xacro (robot description, xacro)
@@ -51,10 +51,4 @@
         mesh_name="link5"
     />
-    <joint name="base_joint" type="fixed">
-        <parent link="world"/>
-        <child link="base_link"/>
-        <origin xyz="0 0 0" rpy="0 0 0"/>
-        <axis xyz="0 0 1"/>
-    </joint>
     <joint name="joint1" type="revolute">
         <origin xyz="0 0 0.06605" rpy="-0.010805 0 0" />
